Commit message: yea

File: description/robot.urdf.xacro (robot description, xacro)
@@ -15,4 +15,4 @@
     <xacro:include filename = "lidar.xacro" />
     <!-- <xacro:include filename = "camera.xacro" /> -->
-    <xacro:include filename = "depth_camera.xacro" />
+   <!--cro:include filename = "depth_camera.xacro" />-->
 </robot>

File: description/robot_main.xacro (robot description, xacro)
@@ -3,4 +3,10 @@
     <xacro:property name="pi" value="3.1415926535897931" />
     <xacro:include filename="inertial_macros.xacro" />
+     <material name="blue">
+      <color rgba="0 0 1 1"/>
+    </material>
+    <material name="black">
+     <color rgba="0 0 0 1"/>
+    </material>
     <!-- Base footprint (ground contact point) -->
     <link name="base_footprint"/>

Commit message: urdf

File: description/robot.urdf.xacro (robot description, xacro)
@@ -1,18 +1,48 @@
+# Create a minimal URDF file
+cat > ~/odin_ws/src/nav2_odin/description/minimal_robot.urdf.xacro << 'EOF'
 <?xml version="1.0"?>
-<robot xmlns:xacro="http://www.ros.org/wiki/xacro"  name="nav2_odin">
-    <xacro:arg name="use_ros2_control"              default="true"/>
-    <xacro:arg name="use_ros2_control_gz_sim"       default="false"/>
-    <!-- Robot_frames -->
-    <xacro:include filename = "robot_main.xacro" />
-    <!-- Controls -->
-    <xacro:if value="$(arg use_ros2_control)">
-        <xacro:include filename = "ros2_control.xacro" />
-    </xacro:if>
-    <xacro:unless value="$(arg use_ros2_control)">
-        <xacro:include filename = "ackermann_drive_control.xacro" />
-    </xacro:unless>
-    <!-- Sensors -->
-    <xacro:include filename = "lidar.xacro" />
-    <!-- <xacro:include filename = "camera.xacro" /> -->
-   <!--cro:include filename = "depth_camera.xacro" />-->
+<robot name="nav2_odin" xmlns:xacro="http://www.ros.org/wiki/xacro">
+  <!-- Base Link -->
+  <link name="base_footprint">
+    <visual>
+      <geometry>
+        <box size="0.3 0.2 0.1"/>
+      </geometry>
+      <material name="blue">
+        <color rgba="0 0 0.8 1"/>
+      </material>
+    </visual>
+  </link>
+  <!-- LiDAR Link -->
+  <link name="lidar_frame">
+    <visual>
+      <geometry>
+        <cylinder length="0.05" radius="0.05"/>
+      </geometry>
+      <material name="red">
+        <color rgba="0.8 0 0 1"/>
+      </material>
+    </visual>
+  </link>
+  <!-- LiDAR Joint -->
+  <joint name="lidar_joint" type="fixed">
+    <parent link="base_footprint"/>
+    <child link="lidar_frame"/>
+    <origin xyz="0 0 0.1" rpy="0 0 0"/>
+  </joint>
+  <!-- Base Link to Odom Transform (static) -->
+  <link name="odom"/>
+  <joint name="odom_joint" type="fixed">
+    <parent link="odom"/>
+    <child link="base_footprint"/>
+    <origin xyz="0 0 0" rpy="0 0 0"/>
+  </joint>
+  <!-- Map to Odom Transform (static) -->
+  <link name="map"/>
+  <joint name="map_joint" type="fixed">
+    <parent link="map"/>
+    <child link="odom"/>
+    <origin xyz="0 0 0" rpy="0 0 0"/>
+  </joint>
 </robot>
+EOF

Commit message: urdf

File: description/robot.urdf.xacro (robot description, xacro)
@@ -1,48 +1,9 @@
-# Create a minimal URDF file
-cat > ~/odin_ws/src/nav2_odin/description/minimal_robot.urdf.xacro << 'EOF'
 <?xml version="1.0"?>
-<robot name="nav2_odin" xmlns:xacro="http://www.ros.org/wiki/xacro">
-  <!-- Base Link -->
-  <link name="base_footprint">
-    <visual>
-      <geometry>
-        <box size="0.3 0.2 0.1"/>
-      </geometry>
-      <material name="blue">
-        <color rgba="0 0 0.8 1"/>
-      </material>
-    </visual>
-  </link>
-  <!-- LiDAR Link -->
-  <link name="lidar_frame">
-    <visual>
-      <geometry>
-        <cylinder length="0.05" radius="0.05"/>
-      </geometry>
-      <material name="red">
-        <color rgba="0.8 0 0 1"/>
-      </material>
-    </visual>
-  </link>
-  <!-- LiDAR Joint -->
-  <joint name="lidar_joint" type="fixed">
-    <parent link="base_footprint"/>
-    <child link="lidar_frame"/>
-    <origin xyz="0 0 0.1" rpy="0 0 0"/>
-  </joint>
-  <!-- Base Link to Odom Transform (static) -->
-  <link name="odom"/>
-  <joint name="odom_joint" type="fixed">
-    <parent link="odom"/>
-    <child link="base_footprint"/>
-    <origin xyz="0 0 0" rpy="0 0 0"/>
-  </joint>
-  <!-- Map to Odom Transform (static) -->
-  <link name="map"/>
-  <joint name="map_joint" type="fixed">
-    <parent link="map"/>
-    <child link="odom"/>
-    <origin xyz="0 0 0" rpy="0 0 0"/>
-  </joint>
+<robot xmlns:xacro="http://www.ros.org/wiki/xacro"  name="robot">
+    <xacro:arg name="use_ros2_control"              default="false"/>
+    <xacro:arg name="use_ros2_control_gz_sim"       default="false"/>
+    <!-- Robot_frames -->
+    <xacro:include filename = "robot_main.xacro" />
+    <!-- Sensors -->
+    <xacro:include filename = "lidar.xacro" />
 </robot>
-EOF
