Commit message: correction

File: description/lidar.xacro (robot description, xacro)
@@ -8,5 +8,5 @@
     <!-- Lidar -->
     <joint name="lidar_joint" type="fixed">
-        <parent link="chasis"/>
+        <parent link="chassis"/>
         <child link="lidar_frame"/>
         <origin xyz="${lidar_offset_x} 0.0 ${lidar_offset_z}" rpy="0 0 ${pi}"/>

File: description/robot_main.xacro (robot description, xacro)
@@ -26,10 +26,4 @@
         </visual>
     </link>
-    <!-- Joint to connect base_link to chasis -->
-    <joint name="base_link_to_chasis" type="fixed">
-        <parent link="base_link"/>
-        <child link="chasis"/>
-        <origin xyz="0 0 0.1" rpy="0 0 0"/>
-    </joint>
     <!-- Front left wheel (steered) -->
     <link name="front_left_wheel">

Commit message: resolve parsing errors

File: description/lidar.xacro (robot description, xacro)
@@ -1,5 +1,4 @@
 <?xml version="1.0"?>
 <robot xmlns:xacro="http://www.ros.org/wiki/xacro" name="robot">
-    <xacro:include filename="inertial_macros.xacro" />
     <xacro:property name="lidar_radius"             value="0.025"/>
     <xacro:property name="lidar_thickness"          value="0.040"/>
@@ -10,5 +9,5 @@
         <parent link="chassis"/>
         <child link="lidar_frame"/>
-        <origin xyz="${lidar_offset_x} 0.0 ${lidar_offset_z}" rpy="0 0 ${pi}"/>
+        <origin xyz="${lidar_offset_x} 0.0 ${lidar_offset_z}" rpy="0 0 3.14159"/> <!-- Replaced pi with 3.14159 -->
     </joint>
     <link name="lidar_frame">
@@ -24,48 +23,4 @@
             </geometry>
         </collision>
-        <xacro:inertial_cylinder mass="0.1" radius="${lidar_radius}" length="${lidar_thickness}">
-            <origin xyz="0 0 0" rpy="0 0 0"/>
-        </xacro:inertial_cylinder>
     </link>
-    <!-- Lidar in gazebo-->
-    <gazebo reference="lidar_frame">
-        <sensor name="lidar" type="gpu_lidar">
-            <gz_frame_id>lidar_frame</gz_frame_id>
-            <pose>0 0 0 0 0 0</pose>
-            <topic>scan</topic>
-            <update_rate>10</update_rate>
-            <always_on>1</always_on>
-            <visualize>true</visualize>
-            <lidar>
-                <scan>
-                    <horizontal>
-                        <samples>360</samples>
-                        <resolution>1</resolution>
-                        <min_angle>-3.14159</min_angle>
-                        <max_angle>3.14159</max_angle>
-                    </horizontal>
-                    <vertical>
-                        <samples>1</samples>
-                        <resolution>0.1</resolution>
-                        <min_angle>0.</min_angle>
-                        <max_angle>0.</max_angle>
-                    </vertical>
-                </scan>
-                <range>
-                    <min>0.08</min>
-                    <max>10.0</max>
-                    <resolution>0.01</resolution>
-                </range>
-                <noise>
-                    <type>gaussian</type>
-                    <mean>0.0</mean>
-                    <stddev>0.01</stddev>
-                </noise>
-            </lidar>
-        <plugin filename="gz-sim-sensors-system"
-                name="gz::sim::systems::Sensors">
-                <render_engine>ogre2</render_engine>
-        </plugin>
-        </sensor>
-    </gazebo>
 </robot>

File: description/robot_main.xacro (robot description, xacro)
@@ -1,9 +1,9 @@
 <?xml version="1.0"?>
 <robot xmlns:xacro="http://www.ros.org/wiki/xacro" name="nav2_odin">
-    <joint name="base_footprint_to_base_link" type="fixed">
-        <parent link="base_footprint"/>
-        <child link="base_link"/>
-        <origin xyz="0 0 0.1" rpy="0 0 0"/>
-    </joint>
+<joint name="base_footprint_to_base_link" type="fixed">
+    <parent link="base_footprint"/>
+    <child link="base_link"/>
+    <origin xyz="0 0 0.1" rpy="0 0 0"/>
+</joint>
     <material name="blue">
         <color rgba="0 0 1 1"/>
@@ -16,4 +16,5 @@
     </material>
     <link name="base_footprint"></link>
+    <!-- Main robot base -->
     <link name="base_link">
         <visual>
@@ -29,4 +30,5 @@
         </collision>
     </link>
+    <!-- Chassis link -->
     <link name="chassis">
         <visual>
@@ -105,5 +107,5 @@
         <parent link="base_link"/>
         <child link="rear_left_wheel"/>
-        <origin xyz="-0.15 0.15 0.05" rpy="pi/2 0 0"/> <!-- Replaced pi/2 with 1.5708 -->
+        <origin xyz="-0.15 0.15 0.05" rpy="1.5708 0 0"/> <!-- Replaced pi/2 with 1.5708 -->
         <axis xyz="0 1 0"/>
     </joint>
@@ -125,5 +127,5 @@
         <parent link="base_link"/>
         <child link="rear_right_wheel"/>
-        <origin xyz="-0.15 -0.15 0.05" rpy="pi/2 0 0"/>
+        <origin xyz="-0.15 -0.15 0.05" rpy="1.5708 0 0"/> <!-- Replaced pi/2 with 1.5708 -->
         <axis xyz="0 1 0"/>
     </joint>
