Commit message: starting to change the entire urdf structure, adapting it for an Ackermann-steering robot

File: description/robot_main.xacro (robot description, xacro)
@@ -2,151 +2,89 @@
 <robot xmlns:xacro="http://www.ros.org/wiki/xacro">
     <xacro:include filename = "inertial_macros.xacro" />
-    <xacro:property name="chassis_length"           value="0.320"/>
-    <xacro:property name="chassis_width"            value="0.240"/>
-    <xacro:property name="chassis_height"           value="0.078"/>
-    <xacro:property name="chassis_mass"             value="0.700"/>
-    <xacro:property name="wheel_radius"             value="0.034"/>
-    <xacro:property name="wheel_thickness"          value="0.026"/>
-    <xacro:property name="wheel_mass"               value="0.050"/>
-    <xacro:property name="wheel_offset_x"           value="0.133"/>
-    <xacro:property name="wheel_offset_y"           value="0.133"/>
-    <xacro:property name="wheel_offset_z"           value="0.020"/>
-    <xacro:property name="caster_wheel_radius"      value="${wheel_radius - wheel_offset_z}"/>
-    <xacro:property name="caster_wheel_mass"        value="0.010"/>
-    <xacro:property name="caster_wheel_offset_x"    value="0.230"/>
-    <xacro:property name="caster_wheel_offset_z"    value="${wheel_offset_z - wheel_radius + caster_wheel_radius}"/>
-    <!-- Colors -->
-    <material name="white">
-        <color rgba= "1 1 1 1"/>
-    </material>
-    <material name="black">
-        <color rgba= "0 0 0 1"/>
-    </material>
-    <material name= "orange">
-        <color rgba= "1 0.25 0 1"/>
-    </material>
-    <material name="cyan">
-        <color rgba= "0 1 1 1"/>
-    </material>
-    <material name="indigo">
-        <color rgba= "0.294 0 0.51 1"/>
-    </material>
-    <!-- convention (except base_link): joint followed by link -->
-    <!-- base_link -->
-    <link name="base_link">
-    </link>
-    <!-- base_footprint -->
-    <joint name="base_footprint_joint" type="fixed">
-        <parent link= "base_link"/>
-        <child link= "base_footprint"/>
-        <origin xyz= "0 0 0" rpy= "0 0 0"/>
-    </joint>
-    <link name="base_footprint">
-    </link>
-    <!-- chasis -->
-    <joint name="chasis_joint" type="fixed">
-        <parent link= "base_link"/>
-        <child link= "chasis"/>
-        <origin xyz= "${-wheel_offset_x} 0 ${-wheel_offset_z}"/>
-    </joint>
-    <link name="chasis">
-        <visual>
-            <origin xyz= "${chassis_length/2} 0 ${chassis_height/2}" rpy= "0 0 0"/>
-            <geometry>
-                <box size = "${chassis_length} ${chassis_width} ${chassis_height}"/>
-            </geometry>
-            <material name= "black"/>
-        </visual>
-        <collision>
-            <origin xyz= "${chassis_length/2} 0 ${chassis_height/2}" rpy= "0 0 0"/>
-            <geometry>
-                <box size = "${chassis_length} ${chassis_width} ${chassis_height}"/>
-            </geometry>
-        </collision>
-        <xacro:inertial_box mass= "0.5" x="${chassis_length}" y="${chassis_width}" z="${chassis_height}">
-            <origin xyz= "${chassis_length/2} 0 ${chassis_height/2}" rpy= "0 0 0"/>
-        </xacro:inertial_box>
-    </link>
-    <gazebo reference="chasis">
-        <material>Gazebo/Black</material>
-    </gazebo>
-    <!-- left_wheel -->
-    <joint name="left_wheel_joint" type="continuous">
-        <parent link= "base_link"/>
-        <child link= "left_wheel"/>
-        <origin xyz= "0 ${wheel_offset_y} 0" rpy = "${pi/2} 0 0"/>
-        <axis xyz= "0 0 -1"/>
-    </joint>
-    <link name="left_wheel">
-        <visual>
-            <geometry>
-                <cylinder radius = "${wheel_radius}" length= "${wheel_thickness}"/>
-            </geometry>
-            <material name= "orange"/>
-        </visual>
-        <collision>
-            <geometry>
-                <sphere radius = "${wheel_radius}" />
-            </geometry>
-        </collision>
-        <xacro:inertial_cylinder mass = "${wheel_mass}" radius= "${wheel_radius}" length= "${wheel_thickness}">
-            <origin xyz= "0 0 0" rpy= "0 0 0"/>
-        </xacro:inertial_cylinder>
-    </link>
-    <gazebo reference="left_wheel">
-        <material>Gazebo/Orange</material>
-    </gazebo>
-    <!-- right_wheel -->
-    <joint name="right_wheel_joint" type="continuous">
-        <parent link= "base_link"/>
-        <child link= "right_wheel"/>
-        <origin xyz= "0 ${-wheel_offset_y} 0" rpy = "${pi/2} 0 0"/>
-        <axis xyz= "0 0 -1"/>
-    </joint>
-    <link name="right_wheel">
-        <visual>
-            <geometry>
-                <cylinder radius = "${wheel_radius}" length= "${wheel_thickness}"/>
-            </geometry>
-            <material name= "orange"/>
-        </visual>
-        <collision>
-            <geometry>
-                <sphere radius = "${wheel_radius}" />
-            </geometry>
-        </collision>
-        <xacro:inertial_cylinder mass = "${wheel_mass}" radius= "${wheel_radius}" length= "${wheel_thickness}">
-            <origin xyz= "0 0 0" rpy= "0 0 0"/>
-        </xacro:inertial_cylinder>
-    </link>
-    <gazebo reference="right_wheel">
-        <material>Gazebo/Orange</material>
-    </gazebo>
-    <!-- caster_wheel -->
-    <joint name="caster_wheel_joint" type="fixed">
-        <parent link= "chasis"/>
-        <child link= "caster_wheel"/>
-        <origin xyz= "${caster_wheel_offset_x} 0 0"/>
-    </joint>
-    <link name="caster_wheel">
-        <visual>
-            <geometry>
-                <sphere radius = "${caster_wheel_radius}"/>
-            </geometry>
-            <material name= "orange"/>
-        </visual>
-        <collision>
-            <geometry>
-                <sphere radius = "${caster_wheel_radius}"/>
-            </geometry>
-        </collision>
-        <xacro:inertial_sphere mass= "${caster_wheel_mass}" radius= "${caster_wheel_radius}">
-            <origin xyz= "0 0 0" rpy= "0 0 0"/>
-        </xacro:inertial_sphere>
-    </link>
-    <gazebo reference="caster_wheel">
-        <material>Gazebo/Orange</material>
-        <mu1 value= "0.0001"/>
-        <mu2 value= "0.0001"/>
-    </gazebo>
+   <?xml version="1.0"?>
+<robot xmlns:xacro="http://www.ros.org/wiki/xacro" name="ackermann_robot">
+  <!-- Base footprint (ground contact point) -->
+  <link name="base_footprint"/>
+  <!-- Main robot base -->
+  <link name="base_link">
+    <visual>
+      <geometry>
+        <box size="0.4 0.3 0.2"/>
+      </geometry>
+      <material name="blue"/>
+    </visual>
+  </link>
+  <!-- Transform from base_footprint to base_link -->
+  <joint name="base_footprint_to_base_link" type="fixed">
+    <parent link="base_footprint"/>
+    <child link="base_link"/>
+    <origin xyz="0 0 0.1" rpy="0 0 0"/>
+  </joint>
+  <!-- Front left wheel (steered) -->
+  <link name="front_left_wheel">
+    <visual>
+      <geometry>
+        <cylinder radius="0.05" length="0.03"/>
+      </geometry>
+      <material name="black"/>
+    </visual>
+  </link>
+  <joint name="front_left_steering_joint" type="continuous">
+    <parent link="base_link"/>
+    <child link="front_left_wheel"/>
+    <origin xyz="0.15 0.15 0.05" rpy="0 0 0"/>
+    <axis xyz="0 0 1"/>
+  </joint>
+  <!-- Front right wheel (steered) -->
+  <link name="front_right_wheel">
+    <visual>
+      <geometry>
+        <cylinder radius="0.05" length="0.03"/>
+      </geometry>
+      <material name="black"/>
+    </visual>
+  </link>
+  <joint name="front_right_steering_joint" type="continuous">
+    <parent link="base_link"/>
+    <child link="front_right_wheel"/>
+    <origin xyz="0.15 -0.15 0.05" rpy="0 0 0"/>
+    <axis xyz="0 0 1"/>
+  </joint>
+  <!-- Rear left wheel (driven) -->
+  <link name="rear_left_wheel">
+    <visual>
+      <geometry>
+        <cylinder radius="0.05" length="0.03"/>
+      </geometry>
+      <material name="black"/>
+    </visual>
+  </link>
+  <joint name="rear_left_wheel_joint" type="continuous">
+    <parent link="base_link"/>
+    <child link="rear_left_wheel"/>
+    <origin xyz="-0.15 0.15 0.05" rpy="${pi/2} 0 0"/>
+    <axis xyz="0 1 0"/>
+  </joint>
+  <!-- Rear right wheel (driven) -->
+  <link name="rear_right_wheel">
+    <visual>
+      <geometry>
+        <cylinder radius="0.05" length="0.03"/>
+      </geometry>
+      <material name="black"/>
+    </visual>
+  </link>
+  <joint name="rear_right_wheel_joint" type="continuous">
+    <parent link="base_link"/>
+    <child link="rear_right_wheel"/>
+    <origin xyz="-0.15 -0.15 0.05" rpy="${pi/2} 0 0"/>
+    <axis xyz="0 1 0"/>
+  </joint>
+  <!-- LiDAR -->
+  <link name="lidar_frame"/>
+  <joint name="base_link_to_lidar" type="fixed">
+    <parent link="base_link"/>
+    <child link="lidar_frame"/>
+    <origin xyz="0.2 0 0.15" rpy="0 0 0"/>
+  </joint>
 </robot>

Commit message: fix robot main, removed sim description file

File: description/robot_main.xacro (robot description, xacro)
@@ -1,90 +1,89 @@
 <?xml version="1.0"?>
-<robot xmlns:xacro="http://www.ros.org/wiki/xacro">
-    <xacro:include filename = "inertial_macros.xacro" />
-   <?xml version="1.0"?>
 <robot xmlns:xacro="http://www.ros.org/wiki/xacro" name="ackermann_robot">
-  <!-- Base footprint (ground contact point) -->
-  <link name="base_footprint"/>
-  <!-- Main robot base -->
-  <link name="base_link">
-    <visual>
-      <geometry>
-        <box size="0.4 0.3 0.2"/>
-      </geometry>
-      <material name="blue"/>
-    </visual>
-  </link>
-  <!-- Transform from base_footprint to base_link -->
-  <joint name="base_footprint_to_base_link" type="fixed">
-    <parent link="base_footprint"/>
-    <child link="base_link"/>
-    <origin xyz="0 0 0.1" rpy="0 0 0"/>
-  </joint>
-  <!-- Front left wheel (steered) -->
-  <link name="front_left_wheel">
-    <visual>
-      <geometry>
-        <cylinder radius="0.05" length="0.03"/>
-      </geometry>
-      <material name="black"/>
-    </visual>
-  </link>
-  <joint name="front_left_steering_joint" type="continuous">
-    <parent link="base_link"/>
-    <child link="front_left_wheel"/>
-    <origin xyz="0.15 0.15 0.05" rpy="0 0 0"/>
-    <axis xyz="0 0 1"/>
-  </joint>
-  <!-- Front right wheel (steered) -->
-  <link name="front_right_wheel">
-    <visual>
-      <geometry>
-        <cylinder radius="0.05" length="0.03"/>
-      </geometry>
-      <material name="black"/>
-    </visual>
-  </link>
-  <joint name="front_right_steering_joint" type="continuous">
-    <parent link="base_link"/>
-    <child link="front_right_wheel"/>
-    <origin xyz="0.15 -0.15 0.05" rpy="0 0 0"/>
-    <axis xyz="0 0 1"/>
-  </joint>
-  <!-- Rear left wheel (driven) -->
-  <link name="rear_left_wheel">
-    <visual>
-      <geometry>
-        <cylinder radius="0.05" length="0.03"/>
-      </geometry>
-      <material name="black"/>
-    </visual>
-  </link>
-  <joint name="rear_left_wheel_joint" type="continuous">
-    <parent link="base_link"/>
-    <child link="rear_left_wheel"/>
-    <origin xyz="-0.15 0.15 0.05" rpy="${pi/2} 0 0"/>
-    <axis xyz="0 1 0"/>
-  </joint>
-  <!-- Rear right wheel (driven) -->
-  <link name="rear_right_wheel">
-    <visual>
-      <geometry>
-        <cylinder radius="0.05" length="0.03"/>
-      </geometry>
-      <material name="black"/>
-    </visual>
-  </link>
-  <joint name="rear_right_wheel_joint" type="continuous">
-    <parent link="base_link"/>
-    <child link="rear_right_wheel"/>
-    <origin xyz="-0.15 -0.15 0.05" rpy="${pi/2} 0 0"/>
-    <axis xyz="0 1 0"/>
-  </joint>
-  <!-- LiDAR -->
-  <link name="lidar_frame"/>
-  <joint name="base_link_to_lidar" type="fixed">
-    <parent link="base_link"/>
-    <child link="lidar_frame"/>
-    <origin xyz="0.2 0 0.15" rpy="0 0 0"/>
-  </joint>
+    <xacro:property name="pi" value="3.1415926535897931" />
+    <xacro:include filename="inertial_macros.xacro" />
+    <!-- Base footprint (ground contact point) -->
+    <link name="base_footprint"/>
+    <!-- Main robot base -->
+    <link name="base_link">
+        <visual>
+            <geometry>
+                <box size="0.4 0.3 0.2"/>
+            </geometry>
+            <material name="blue"/>
+        </visual>
+    </link>
+    <!-- Transform from base_footprint to base_link -->
+    <joint name="base_footprint_to_base_link" type="fixed">
+        <parent link="base_footprint"/>
+        <child link="base_link"/>
+        <origin xyz="0 0 0.1" rpy="0 0 0"/>
+    </joint>
+    <!-- Front left wheel (steered) -->
+    <link name="front_left_wheel">
+        <visual>
+            <geometry>
+                <cylinder radius="0.05" length="0.03"/>
+            </geometry>
+            <material name="black"/>
+        </visual>
+    </link>
+    <joint name="front_left_steering_joint" type="continuous">
+        <parent link="base_link"/>
+        <child link="front_left_wheel"/>
+        <origin xyz="0.15 0.15 0.05" rpy="0 0 0"/>
+        <axis xyz="0 0 1"/>
+    </joint>
+    <!-- Front right wheel (steered) -->
+    <link name="front_right_wheel">
+        <visual>
+            <geometry>
+                <cylinder radius="0.05" length="0.03"/>
+            </geometry>
+            <material name="black"/>
+        </visual>
+    </link>
+    <joint name="front_right_steering_joint" type="continuous">
+        <parent link="base_link"/>
+        <child link="front_right_wheel"/>
+        <origin xyz="0.15 -0.15 0.05" rpy="0 0 0"/>
+        <axis xyz="0 0 1"/>
+    </joint>
+    <!-- Rear left wheel (driven) -->
+    <link name="rear_left_wheel">
+        <visual>
+            <geometry>
+                <cylinder radius="0.05" length="0.03"/>
+            </geometry>
+            <material name="black"/>
+        </visual>
+    </link>
+    <joint name="rear_left_wheel_joint" type="continuous">
+        <parent link="base_link"/>
+        <child link="rear_left_wheel"/>
+        <origin xyz="-0.15 0.15 0.05" rpy="${pi/2} 0 0"/>
+        <axis xyz="0 1 0"/>
+    </joint>
+    <!-- Rear right wheel (driven) -->
+    <link name="rear_right_wheel">
+        <visual>
+            <geometry>
+                <cylinder radius="0.05" length="0.03"/>
+            </geometry>
+            <material name="black"/>
+        </visual>
+    </link>
+    <joint name="rear_right_wheel_joint" type="continuous">
+        <parent link="base_link"/>
+        <child link="rear_right_wheel"/>
+        <origin xyz="-0.15 -0.15 0.05" rpy="${pi/2} 0 0"/>
+        <axis xyz="0 1 0"/>
+    </joint>
+    <!-- LiDAR -->
+    <link name="lidar_frame"/>
+    <joint name="base_link_to_lidar" type="fixed">
+        <parent link="base_link"/>
+        <child link="lidar_frame"/>
+        <origin xyz="0.2 0 0.15" rpy="0 0 0"/>
+    </joint>
 </robot>

Commit message: main

File: description/robot_main.xacro (robot description, xacro)
@@ -1,5 +1,5 @@
 <?xml version="1.0"?>
 <robot xmlns:xacro="http://www.ros.org/wiki/xacro" name="ackermann_robot">
-    <xacro:property name="pi" value="3.1415926535897931" />
+    <origin xyz="0 0 0" rpy="${pi/2} 0 0" />
     <xacro:include filename="inertial_macros.xacro" />
      <material name="blue">

Commit message: fix lidarframe

File: description/robot_main.xacro (robot description, xacro)
@@ -86,10 +86,2 @@
         <axis xyz="0 1 0"/>
     </joint>
-    <!-- LiDAR -->
-    <link name="lidar_frame"/>
-    <joint name="base_link_to_lidar" type="fixed">
-        <parent link="base_link"/>
-        <child link="lidar_frame"/>
-        <origin xyz="0.2 0 0.15" rpy="0 0 0"/>
-    </joint>
-</robot>

Commit message: fixed robot_main

File: description/robot_main.xacro (robot description, xacro)
@@ -1,14 +1,18 @@
 <?xml version="1.0"?>
 <robot xmlns:xacro="http://www.ros.org/wiki/xacro" name="ackermann_robot">
-    <origin xyz="0 0 0" rpy="${pi/2} 0 0" />
     <xacro:include filename="inertial_macros.xacro" />
-     <material name="blue">
-      <color rgba="0 0 1 1"/>
+    <material name="blue">
+        <color rgba="0 0 1 1"/>
     </material>
     <material name="black">
-     <color rgba="0 0 0 1"/>
+        <color rgba="0 0 0 1"/>
     </material>
     <!-- Base footprint (ground contact point) -->
-    <link name="base_footprint"/>
+    <link name="base_footprint">
+        <inertial>
+            <mass value="0.001"/>
+            <inertia ixx="0.001" ixy="0.0" ixz="0.0" iyy="0.001" iyz="0.0" izz="0.001"/>
+        </inertial>
+    </link>
     <!-- Main robot base -->
     <link name="base_link">
@@ -19,4 +23,8 @@
             <material name="blue"/>
         </visual>
+        <inertial>
+            <mass value="5.0"/>
+            <inertia ixx="0.1" ixy="0.0" ixz="0.0" iyy="0.1" iyz="0.0" izz="0.1"/>
+        </inertial>
     </link>
     <!-- Transform from base_footprint to base_link -->
@@ -34,4 +42,8 @@
             <material name="black"/>
         </visual>
+        <inertial>
+            <mass value="0.5"/>
+            <inertia ixx="0.001" ixy="0.0" ixz="0.0" iyy="0.001" iyz="0.0" izz="0.001"/>
+        </inertial>
     </link>
     <joint name="front_left_steering_joint" type="continuous">
@@ -49,4 +61,8 @@
             <material name="black"/>
         </visual>
+        <inertial>
+            <mass value="0.5"/>
+            <inertia ixx="0.001" ixy="0.0" ixz="0.0" iyy="0.001" iyz="0.0" izz="0.001"/>
+        </inertial>
     </link>
     <joint name="front_right_steering_joint" type="continuous">
@@ -64,4 +80,8 @@
             <material name="black"/>
         </visual>
+        <inertial>
+            <mass value="0.5"/>
+            <inertia ixx="0.001" ixy="0.0" ixz="0.0" iyy="0.001" iyz="0.0" izz="0.001"/>
+        </inertial>
     </link>
     <joint name="rear_left_wheel_joint" type="continuous">
@@ -79,4 +99,8 @@
             <material name="black"/>
         </visual>
+        <inertial>
+            <mass value="0.5"/>
+            <inertia ixx="0.001" ixy="0.0" ixz="0.0" iyy="0.001" iyz="0.0" izz="0.001"/>
+        </inertial>
     </link>
     <joint name="rear_right_wheel_joint" type="continuous">
@@ -86,2 +110,3 @@
         <axis xyz="0 1 0"/>
     </joint>
+</robot>

Commit message: fixed robot main

File: description/robot_main.xacro (robot description, xacro)
@@ -7,4 +7,7 @@
     <material name="black">
         <color rgba="0 0 0 1"/>
+    </material>
+    <material name="orange">
+        <color rgba="1 0.5 0 1"/>
     </material>
     <!-- Base footprint (ground contact point) -->
@@ -32,4 +35,23 @@
         <parent link="base_footprint"/>
         <child link="base_link"/>
+        <origin xyz="0 0 0.1" rpy="0 0 0"/>
+    </joint>
+    <!-- Chasis link -->
+    <link name="chasis">
+        <visual>
+            <geometry>
+                <box size="0.3 0.2 0.1"/>
+            </geometry>
+            <material name="blue"/>
+        </visual>
+        <inertial>
+            <mass value="2.0"/>
+            <inertia ixx="0.01" ixy="0.0" ixz="0.0" iyy="0.01" iyz="0.0" izz="0.01"/>
+        </inertial>
+    </link>
+    <!-- Joint to connect base_link to chasis -->
+    <joint name="base_link_to_chasis" type="fixed">
+        <parent link="base_link"/>
+        <child link="chasis"/>
         <origin xyz="0 0 0.1" rpy="0 0 0"/>
     </joint>

Commit message: changed from mppi to DWb for more stability and avoiding package errors

File: description/robot_main.xacro (robot description, xacro)
@@ -14,6 +14,6 @@
     <link name="base_footprint">
         <inertial>
-            <mass value="0.001"/>
-            <inertia ixx="0.001" ixy="0.0" ixz="0.0" iyy="0.001" iyz="0.0" izz="0.001"/>
+            <mass value="0.00"/>
+            <inertia ixx="0.00" ixy="0.0" ixz="0.0" iyy="0.00" iyz="0.0" izz="0.00"/>
         </inertial>
     </link>
@@ -132,3 +132,15 @@
         <axis xyz="0 1 0"/>
     </joint>
+        <link name="base_dummy">
+    <inertial>
+        <mass value="0.001"/>
+        <origin xyz="0 0 0"/>
+        <inertia ixx="0.001" ixy="0.0" ixz="0.0" iyy="0.001" iyz="0.0" izz="0.001"/>
+    </inertial>
+    </link>
+    <joint name="base_dummy_joint" type="fixed">
+    <parent link="base_dummy"/>
+    <child link="base_footprint"/>
+    <origin xyz="0 0 0" rpy="0 0 0"/>
+    </joint>
 </robot>

Commit message: ya

File: description/robot_main.xacro (robot description, xacro)
@@ -132,5 +132,5 @@
         <axis xyz="0 1 0"/>
     </joint>
-        <link name="base_dummy">
+    <link name="base_dummy">
     <inertial>
         <mass value="0.001"/>

Commit message: yah

File: description/robot_main.xacro (robot description, xacro)
@@ -136,5 +136,5 @@
         <mass value="0.001"/>
         <origin xyz="0 0 0"/>
-        <inertia ixx="0.001" ixy="0.0" ixz="0.0" iyy="0.001" iyz="0.0" izz="0.001"/>
+        <inertia ixx="0.00" ixy="0.0" ixz="0.0" iyy="0.00" iyz="0.0" izz="0.00"/>
     </inertial>
     </link>

Commit message: j

File: description/robot_main.xacro (robot description, xacro)
@@ -134,5 +134,5 @@
     <link name="base_dummy">
     <inertial>
-        <mass value="0.001"/>
+        <mass value="0.00"/>
         <origin xyz="0 0 0"/>
         <inertia ixx="0.00" ixy="0.0" ixz="0.0" iyy="0.00" iyz="0.0" izz="0.00"/>

Commit message: fixed steering_node, espserial, robot.launch

File: description/robot_main.xacro (robot description, xacro)
@@ -14,6 +14,6 @@
     <link name="base_footprint">
         <inertial>
-            <mass value="0.00"/>
-            <inertia ixx="0.00" ixy="0.0" ixz="0.0" iyy="0.00" iyz="0.0" izz="0.00"/>
+            <mass value="0.001"/>
+            <inertia ixx="0.001" ixy="0.0" ixz="0.0" iyy="0.001" iyz="0.0" izz="0.001"/>
         </inertial>
     </link>
@@ -132,15 +132,3 @@
         <axis xyz="0 1 0"/>
     </joint>
-    <link name="base_dummy">
-    <inertial>
-        <mass value="0.00"/>
-        <origin xyz="0 0 0"/>
-        <inertia ixx="0.00" ixy="0.0" ixz="0.0" iyy="0.00" iyz="0.0" izz="0.00"/>
-    </inertial>
-    </link>
-    <joint name="base_dummy_joint" type="fixed">
-    <parent link="base_dummy"/>
-    <child link="base_footprint"/>
-    <origin xyz="0 0 0" rpy="0 0 0"/>
-    </joint>
 </robot>

Commit message: please work

File: description/robot_main.xacro (robot description, xacro)
@@ -1,5 +1,4 @@
 <?xml version="1.0"?>
 <robot xmlns:xacro="http://www.ros.org/wiki/xacro" name="nav2_odin">
-    <xacro:include filename="inertial_macros.xacro" />
     <material name="blue">
         <color rgba="0 0 1 1"/>
@@ -131,4 +130,16 @@
         <origin xyz="-0.15 -0.15 0.05" rpy="${pi/2} 0 0"/>
         <axis xyz="0 1 0"/>
+        </joint>
+    <link name="base_dummy_inertialless">
+        <visual>
+            <geometry>
+                <box size="0.01 0.01 0.01"/>
+            </geometry>
+        </visual>
+    </link>
+    <joint name="base_dummy_joint" type="fixed">
+        <parent link="base_dummy_inertialless"/>
+        <child link="base_dummy"/>
+        <origin xyz="0 0 0" rpy="0 0 0"/>
     </joint>
 </robot>
