Commit message: optimized code

File: description/robot_main.xacro (robot description, xacro)
@@ -1,4 +1,5 @@
 <?xml version="1.0"?>
 <robot xmlns:xacro="http://www.ros.org/wiki/xacro" name="nav2_odin">
+    <xacro:include filename="inertial_macros.xacro" />
     <material name="blue">
         <color rgba="0 0 1 1"/>
@@ -130,16 +131,6 @@
         <origin xyz="-0.15 -0.15 0.05" rpy="${pi/2} 0 0"/>
         <axis xyz="0 1 0"/>
-        </joint>
-    <link name="base_dummy_inertialless">
-        <visual>
-            <geometry>
-                <box size="0.01 0.01 0.01"/>
-            </geometry>
-        </visual>
-    </link>
-    <joint name="base_dummy_joint" type="fixed">
-        <parent link="base_dummy_inertialless"/>
-        <child link="base_dummy"/>
-        <origin xyz="0 0 0" rpy="0 0 0"/>
     </joint>
+    <!-- Remove base_dummy completely as it's not needed -->
+    <!-- The root should be base_footprint -->
 </robot>

Commit message: removed inertia

File: description/robot_main.xacro (robot description, xacro)
@@ -11,11 +11,5 @@
         <color rgba="1 0.5 0 1"/>
     </material>
-    <!-- Base footprint (ground contact point) -->
-    <link name="base_footprint">
-        <inertial>
-            <mass value="0.001"/>
-            <inertia ixx="0.001" ixy="0.0" ixz="0.0" iyy="0.001" iyz="0.0" izz="0.001"/>
-        </inertial>
-    </link>
+    <link name="base_footprint"></link>
     <!-- Main robot base -->
     <link name="base_link">
@@ -26,8 +20,4 @@
             <material name="blue"/>
         </visual>
-        <inertial>
-            <mass value="5.0"/>
-            <inertia ixx="0.1" ixy="0.0" ixz="0.0" iyy="0.1" iyz="0.0" izz="0.1"/>
-        </inertial>
     </link>
     <!-- Transform from base_footprint to base_link -->
@@ -45,8 +35,4 @@
             <material name="blue"/>
         </visual>
-        <inertial>
-            <mass value="2.0"/>
-            <inertia ixx="0.01" ixy="0.0" ixz="0.0" iyy="0.01" iyz="0.0" izz="0.01"/>
-        </inertial>
     </link>
     <!-- Joint to connect base_link to chasis -->
@@ -64,8 +50,4 @@
             <material name="black"/>
         </visual>
-        <inertial>
-            <mass value="0.5"/>
-            <inertia ixx="0.001" ixy="0.0" ixz="0.0" iyy="0.001" iyz="0.0" izz="0.001"/>
-        </inertial>
     </link>
     <joint name="front_left_steering_joint" type="continuous">
@@ -83,8 +65,4 @@
             <material name="black"/>
         </visual>
-        <inertial>
-            <mass value="0.5"/>
-            <inertia ixx="0.001" ixy="0.0" ixz="0.0" iyy="0.001" iyz="0.0" izz="0.001"/>
-        </inertial>
     </link>
     <joint name="front_right_steering_joint" type="continuous">
@@ -102,8 +80,4 @@
             <material name="black"/>
         </visual>
-        <inertial>
-            <mass value="0.5"/>
-            <inertia ixx="0.001" ixy="0.0" ixz="0.0" iyy="0.001" iyz="0.0" izz="0.001"/>
-        </inertial>
     </link>
     <joint name="rear_left_wheel_joint" type="continuous">
@@ -121,8 +95,4 @@
             <material name="black"/>
         </visual>
-        <inertial>
-            <mass value="0.5"/>
-            <inertia ixx="0.001" ixy="0.0" ixz="0.0" iyy="0.001" iyz="0.0" izz="0.001"/>
-        </inertial>
     </link>
     <joint name="rear_right_wheel_joint" type="continuous">
@@ -132,5 +102,3 @@
         <axis xyz="0 1 0"/>
     </joint>
-    <!-- Remove base_dummy completely as it's not needed -->
-    <!-- The root should be base_footprint -->
 </robot>

Commit message: footprint to base tf, added pi xacro property, added slamtoolbox on lifecyclenode,  added static tf node

File: description/robot_main.xacro (robot description, xacro)
@@ -2,4 +2,10 @@
 <robot xmlns:xacro="http://www.ros.org/wiki/xacro" name="nav2_odin">
     <xacro:include filename="inertial_macros.xacro" />
+<xacro:property name="pi" value="3.1415926535897931" />
+<joint name="base_footprint_to_base_link" type="fixed">
+    <parent link="base_footprint"/>
+    <child link="base_link"/>
+    <origin xyz="0 0 0.1" rpy="0 0 0"/>
+</joint>
     <material name="blue">
         <color rgba="0 0 1 1"/>

Commit message: removed pi value

File: description/robot_main.xacro (robot description, xacro)
@@ -2,5 +2,4 @@
 <robot xmlns:xacro="http://www.ros.org/wiki/xacro" name="nav2_odin">
     <xacro:include filename="inertial_macros.xacro" />
-<xacro:property name="pi" value="3.1415926535897931" />
 <joint name="base_footprint_to_base_link" type="fixed">
     <parent link="base_footprint"/>

Commit message: fixing a duplicate

File: description/robot_main.xacro (robot description, xacro)
@@ -22,19 +22,4 @@
             <geometry>
                 <box size="0.4 0.3 0.2"/>
-            </geometry>
-            <material name="blue"/>
-        </visual>
-    </link>
-    <!-- Transform from base_footprint to base_link -->
-    <joint name="base_footprint_to_base_link" type="fixed">
-        <parent link="base_footprint"/>
-        <child link="base_link"/>
-        <origin xyz="0 0 0.1" rpy="0 0 0"/>
-    </joint>
-    <!-- Chasis link -->
-    <link name="chasis">
-        <visual>
-            <geometry>
-                <box size="0.3 0.2 0.1"/>
             </geometry>
             <material name="blue"/>

Commit message: new robot.main

File: description/robot_main.xacro (robot description, xacro)
@@ -1,10 +1,9 @@
 <?xml version="1.0"?>
 <robot xmlns:xacro="http://www.ros.org/wiki/xacro" name="nav2_odin">
-    <xacro:include filename="inertial_macros.xacro" />
-<joint name="base_footprint_to_base_link" type="fixed">
-    <parent link="base_footprint"/>
-    <child link="base_link"/>
-    <origin xyz="0 0 0.1" rpy="0 0 0"/>
-</joint>
+    <joint name="base_footprint_to_base_link" type="fixed">
+        <parent link="base_footprint"/>
+        <child link="base_link"/>
+        <origin xyz="0 0 0.1" rpy="0 0 0"/>
+    </joint>
     <material name="blue">
         <color rgba="0 0 1 1"/>
@@ -17,5 +16,4 @@
     </material>
     <link name="base_footprint"></link>
-    <!-- Main robot base -->
     <link name="base_link">
         <visual>
@@ -25,5 +23,29 @@
             <material name="blue"/>
         </visual>
+        <collision>
+            <geometry>
+                <box size="0.4 0.3 0.2"/>
+            </geometry>
+        </collision>
     </link>
+    <link name="chassis">
+        <visual>
+            <geometry>
+                <box size="0.35 0.25 0.05"/>
+            </geometry>
+            <material name="blue"/>
+        </visual>
+        <collision>
+            <geometry>
+                <box size="0.35 0.25 0.05"/>
+            </geometry>
+        </collision>
+    </link>
+    <!-- Joint to connect base_link to chassis -->
+    <joint name="base_link_to_chassis" type="fixed">
+        <parent link="base_link"/>
+        <child link="chassis"/>
+        <origin xyz="0 0 0.125" rpy="0 0 0"/>
+    </joint>
     <!-- Front left wheel (steered) -->
     <link name="front_left_wheel">
@@ -34,4 +56,9 @@
             <material name="black"/>
         </visual>
+        <collision>
+            <geometry>
+                <cylinder radius="0.05" length="0.03"/>
+            </geometry>
+        </collision>
     </link>
     <joint name="front_left_steering_joint" type="continuous">
@@ -49,4 +76,9 @@
             <material name="black"/>
         </visual>
+        <collision>
+            <geometry>
+                <cylinder radius="0.05" length="0.03"/>
+            </geometry>
+        </collision>
     </link>
     <joint name="front_right_steering_joint" type="continuous">
@@ -64,9 +96,14 @@
             <material name="black"/>
         </visual>
+        <collision>
+            <geometry>
+                <cylinder radius="0.05" length="0.03"/>
+            </geometry>
+        </collision>
     </link>
     <joint name="rear_left_wheel_joint" type="continuous">
         <parent link="base_link"/>
         <child link="rear_left_wheel"/>
-        <origin xyz="-0.15 0.15 0.05" rpy="${pi/2} 0 0"/>
+        <origin xyz="-0.15 0.15 0.05" rpy="pi/2 0 0"/> <!-- Replaced pi/2 with 1.5708 -->
         <axis xyz="0 1 0"/>
     </joint>
@@ -79,9 +116,14 @@
             <material name="black"/>
         </visual>
+        <collision>
+            <geometry>
+                <cylinder radius="0.05" length="0.03"/>
+            </geometry>
+        </collision>
     </link>
     <joint name="rear_right_wheel_joint" type="continuous">
         <parent link="base_link"/>
         <child link="rear_right_wheel"/>
-        <origin xyz="-0.15 -0.15 0.05" rpy="${pi/2} 0 0"/>
+        <origin xyz="-0.15 -0.15 0.05" rpy="pi/2 0 0"/>
         <axis xyz="0 1 0"/>
     </joint>

Commit message: mapper

File: description/robot_main.xacro (robot description, xacro)
@@ -130,3 +130,8 @@
         <axis xyz="0 1 0"/>
     </joint>
+    <joint name="lidar_joint" type="fixed">
+    <parent link="chassis"/>
+    <child link="lidar_frame"/>
+    <origin xyz="${lidar_offset_x} 0.0 ${lidar_offset_z}" rpy="0 0 3.14159"/>
+    </joint>
 </robot>

Commit message: ADDED TF STATIC., corrextion if robotmain

File: description/robot_main.xacro (robot description, xacro)
@@ -1,10 +1,13 @@
 <?xml version="1.0"?>
 <robot xmlns:xacro="http://www.ros.org/wiki/xacro" name="nav2_odin">
-    <xacro:include filename = "lidar.xacro" />
-<joint name="base_footprint_to_base_link" type="fixed">
-    <parent link="base_footprint"/>
-    <child link="base_link"/>
-    <origin xyz="0 0 0.1" rpy="0 0 0"/>
-</joint>
+    <xacro:include filename="lidar.xacro" />
+    <!-- Define lidar properties here since they're used in this file -->
+    <xacro:property name="lidar_offset_x" value="0.230"/>
+    <xacro:property name="lidar_offset_z" value="0.098"/>
+    <joint name="base_footprint_to_base_link" type="fixed">
+        <parent link="base_footprint"/>
+        <child link="base_link"/>
+        <origin xyz="0 0 0.1" rpy="0 0 0"/>
+    </joint>
     <material name="blue">
         <color rgba="0 0 1 1"/>
@@ -131,8 +134,3 @@
         <axis xyz="0 1 0"/>
     </joint>
-    <joint name="lidar_joint" type="fixed">
-    <parent link="chassis"/>
-    <child link="lidar_frame"/>
-    <origin xyz="${lidar_offset_x} 0.0 ${lidar_offset_z}" rpy="0 0 3.14159"/>
-    </joint>
 </robot>
